File: Rev2/BaseBoard/BaseBoard.kicad_pcb (KiCad board)
At the start: 2 copper layers, 88 x 79 mm, 86 parts, among them J1 Barrel_Jack_MountingPin, J2 WS2812B CON, J3 MIC CON, J4 SJ1-3523N, J5 SJ1-3523N, J6 PASSIVE 5V LED CON, J7 JTAG CON, J8 UART CON, J9 OLED, Q1 BC618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

Commit message: Finished rev 2
Parts:
- TP11, TP12, TP2, TP3, TP9: moved to F.Cu
- moved C2 15.8 mm to (114.2, 74.8), turned to -90 degrees
- moved TP1 14.6 mm to (127.0, 71.0)
- moved TP2 14.4 mm to (118.8, 73.8), turned to 0 degrees
- moved U1 12.3 mm to (106.7, 77.3)
- moved U2 9.71 mm to (106.7, 88.2)
- moved TP7 9.29 mm to (168.8, 118.8)
- moved D5 9.20 mm to (131.8, 90.8), turned to 90 degrees
- moved TP5 8.43 mm to (173.2, 100.8)
- moved TP12 7.75 mm to (139.0, 82.2), turned to 0 degrees
- moved TP10 6.71 mm to (141.0, 76.0)
- moved TP11 6.25 mm to (136.0, 93.8), turned to 0 degrees
- moved D6 6.24 mm to (135.8, 80.7), turned to -90 degrees
- moved TP3 5.37 mm to (110.5, 83.8), turned to 0 degrees
- moved C14 3.56 mm to (144.0, 100.0), turned to 0 degrees
- moved C19 3.52 mm to (126.5, 80.5), turned to 0 degrees
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- renumbered PB_0 to PB0, PB_1 to PB1
Connections:
- R19 pad 2: /InputPeripherals/I2C_SDA -> /I2C_SDA_EXT
- R20 pad 2: /InputPeripherals/I2C_SCL -> /I2C_SCL_EXT
Routing:
- net GND: track 0.00 -> 1275.8 mm, vias 0 -> 34
- net +3V3: track 0.00 -> 676.2 mm, vias 0 -> 5
- net -3V3: track 0.00 -> 226.1 mm, vias 0 -> 6
- net /InputPeripherals/MUX_A: track 0.00 -> 98.9 mm, vias 0 -> 6
- net /I2C_SCL_EXT: track 0.00 -> 98.3 mm, vias 0 -> 5
- net /OutputPeripherals/SIG_ACTIVE_LED: track 0.00 -> 85.8 mm, vias 0 -> 4
- net /InputPeripherals/MUX_B: track 0.00 -> 83.0 mm, vias 0 -> 4
- net /I2C_SDA_EXT: track 0.00 -> 75.4 mm, vias 0 -> 5
- net Net-(U1-VI): track 0.00 -> 63.9 mm
- net /JTAG_TDI: track 0.00 -> 61.8 mm, vias 0 -> 3
- net /InputPeripherals/PB_0: track 0.00 -> 60.0 mm, vias 0 -> 5
- net /InputPeripherals/AUX_IN_R: track 0.00 -> 59.9 mm, vias 0 -> 2
- net /InputPeripherals/PB_1: track 0.00 -> 53.1 mm, vias 0 -> 6
- net /JTAG_TCK: track 0.00 -> 52.4 mm, vias 0 -> 1
- net /JTAG_TMS: track 0.00 -> 52.3 mm, vias 0 -> 1
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Other:
- outline, holes or cut-outs redrawn
- board text added: "AA filter"
- board text added: "SP filter"
